File: examples/STM32/displays/oled-096-1/cabling/Cabling.kicad_sch (KiCad schematic)
At the start: 2 parts, among them J1 Conn_01x04, U1 NUCLEO144-F767ZI

Commit message: updates
Connections:
- net +3.3V: now also J1.2 (Pin_2)
- net GND: now also J1.1 (Pin_1)
- net SCL: now also J1.3 (Pin_3)
- net SDA: now also J1.4 (Pin_4)
Changed lines of the file:
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@@
+	(wire
+		(pts
+			(xy 256.54 55.88) (xy 261.62 55.88)
+		)
+		(stroke
+			(width 0)
+			(type default)
+		)
+	)
+	(wire
+		(pts
+			(xy 256.54 53.34) (xy 261.62 53.34)
+		)
+		(stroke
+			(width 0)
+			(type default)
+		)
+	)
+	(wire
+		(pts
+			(xy 256.54 48.26) (xy 261.62 48.26)
+		)
+		(stroke
+			(width 0)
+			(type default)
+		)
+	)
 	(wire
 		(pts
@@
 	(wire
 		(pts
+			(xy 256.54 50.8) (xy 261.62 50.8)
+		)
+		(stroke
+			(width 0)
+			(type default)
+		)
+	)
+	(wire
+		(pts
 			(xy 311.15 20.32) (xy 311.15 26.67)
 		)
@@
 	)
 	(label "GND"
-		(at 261.62 55.88 0)
+		(at 261.62 48.26 0)
 		(fields_autoplaced yes)
 		(effects
@@
 	)
 	(label "SDA"
-		(at 261.62 50.8 0)
+		(at 261.62 55.88 0)
 		(fields_autoplaced yes)
 		(effects
@@
 	)
 	(label "+3.3V"
-		(at 261.62 48.26 0)
+		(at 261.62 50.8 0)
 		(fields_autoplaced yes)
 		(effects
